Commit message: feat: add collision and inertial properties to robot model

File: ros2_ws/src/robot_description/urdf/common_macros.xacro (robot description, xacro)
@@ -1,9 +1,12 @@
 <?xml version="1.0"?>
 <robot xmlns:xacro="http://www.ros.org/wiki/xacro">
-  <!-- 长方体 Link 模板 -->
+  <!-- ========================= -->
+  <!-- Box Link Macro -->
+  <!-- ========================= -->
   <xacro:macro
     name="box_link"
-    params="name size_x size_y size_z origin_xyz color">
+    params="name size_x size_y size_z origin_xyz color mass">
     <link name="${name}">
+      <!-- Visual -->
       <visual>
         <origin
@@ -18,7 +21,37 @@
         </material>
       </visual>
+      <!-- Collision -->
+      <collision>
+        <origin
+          xyz="${origin_xyz}"
+          rpy="0 0 0"
+        />
+        <geometry>
+          <box size="${size_x} ${size_y} ${size_z}"/>
+        </geometry>
+      </collision>
+<inertial>
+  <!-- 质心和几何中心保持一致 -->
+  <origin
+    xyz="${origin_xyz}"
+    rpy="0 0 0"
+  />
+  <!-- 质量 -->
+  <mass value="${mass}"/>
+  <!-- 长方体惯性矩阵 -->
+  <inertia
+    ixx="${mass / 12.0 * (size_y * size_y + size_z * size_z)}"
+    ixy="0.0"
+    ixz="0.0"
+    iyy="${mass / 12.0 * (size_x * size_x + size_z * size_z)}"
+    iyz="0.0"
+    izz="${mass / 12.0 * (size_x * size_x + size_y * size_y)}"
+  />
+</inertial>
     </link>
   </xacro:macro>
-  <!-- 旋转关节模板 -->
+  <!-- ========================= -->
+  <!-- Revolute Joint Macro -->
+  <!-- ========================= -->
   <xacro:macro
     name="revolute_joint"

File: ros2_ws/src/robot_description/urdf/simple_arm.urdf.xacro (robot description, xacro)
@@ -27,4 +27,5 @@
     origin_xyz="0 0 ${base_height / 2.0}"
     color="0.6 0.6 0.6 1.0"
+    mass="5.0"
   />
   <!-- link1 -->
@@ -36,4 +37,5 @@
     origin_xyz="0 0 ${link1_length / 2.0}"
     color="0.2 0.4 0.8 1.0"
+     mass="2.0"
   />
   <!-- joint1 -->
@@ -55,4 +57,5 @@
     origin_xyz="${link2_length / 2.0} 0 0"
     color="1.0 0.5 0.1 1.0"
+     mass="1.0"
   />
   <!-- joint2 -->
