Commit message: add complete 6dof robot model

File: ros2_ws/src/simple_6dof_description/urdf/simple_6dof_arm.urdf.xacro (robot description, xacro)
@@ -2,65 +2,155 @@
 <robot xmlns:xacro="http://www.ros.org/wiki/xacro"
        name="simple_6dof_arm">
-    <!-- ===================== -->
-    <!-- Base -->
-    <!-- ===================== -->
-    <link name="base_link">
-        <visual>
-            <geometry>
-                <box size="0.3 0.3 0.1"/>
-            </geometry>
-            <origin xyz="0 0 0"/>
-        </visual>
-    </link>
-    <!-- ===================== -->
-    <!-- Joint 1 : Base rotate -->
-    <!-- ===================== -->
-    <joint name="joint1"
-           type="revolute">
-        <parent link="base_link"/>
-        <child link="link1"/>
-        <origin xyz="0 0 0.1"
-                rpy="0 0 0"/>
-        <!-- 绕Z轴旋转 -->
-        <axis xyz="0 0 1"/>
-        <limit
-            lower="-3.14"
-            upper="3.14"
-            effort="10"
-            velocity="1"/>
-    </joint>
-    <link name="link1">
-        <visual>
-            <geometry>
-                <cylinder radius="0.05"
-                          length="0.3"/>
-            </geometry>
-            <origin xyz="0 0 0.15"/>
-        </visual>
-    </link>
-    <!-- ===================== -->
-    <!-- Joint 2 : Shoulder -->
-    <!-- ===================== -->
-    <joint name="joint2"
-           type="revolute">
-        <parent link="link1"/>
-        <child link="link2"/>
-        <origin xyz="0 0 0.3"
-                rpy="0 0 0"/>
-        <!-- 绕Y轴旋转 -->
-        <axis xyz="0 1 0"/>
-        <limit
-            lower="-1.57"
-            upper="1.57"
-            effort="10"
-            velocity="1"/>
-    </joint>
-   <link name="link2">
+<!-- ===================== -->
+<!-- Base -->
+<!-- ===================== -->
+<link name="base_link">
     <visual>
         <geometry>
-            <box size="0.3 0.08 0.08"/>
+            <box size="0.3 0.3 0.1"/>
+        </geometry>
+        <origin xyz="0 0 0"/>
+    </visual>
+</link>
+<!-- ===================== -->
+<!-- Joint 1 Base Rotation -->
+<!-- ===================== -->
+<joint name="joint1"
+       type="revolute">
+    <parent link="base_link"/>
+    <child link="link1"/>
+    <origin xyz="0 0 0.1"/>
+    <axis xyz="0 0 1"/>
+    <limit
+        lower="-3.14"
+        upper="3.14"
+        effort="20"
+        velocity="1"/>
+</joint>
+<link name="link1">
+    <visual>
+        <geometry>
+            <cylinder radius="0.05"
+                      length="0.35"/>
+        </geometry>
+        <origin xyz="0 0 0.175"/>
+    </visual>
+</link>
+<!-- ===================== -->
+<!-- Joint 2 Shoulder -->
+<!-- ===================== -->
+<joint name="joint2"
+       type="revolute">
+    <parent link="link1"/>
+    <child link="link2"/>
+    <origin xyz="0 0 0.35"/>
+    <axis xyz="0 1 0"/>
+    <limit
+        lower="-1.8"
+        upper="1.8"
+        effort="20"
+        velocity="1"/>
+</joint>
+<link name="link2">
+    <visual>
+        <geometry>
+            <box size="0.35 0.08 0.08"/>
+        </geometry>
+        <origin xyz="0.175 0 0"/>
+    </visual>
+</link>
+<!-- ===================== -->
+<!-- Joint 3 Elbow -->
+<!-- ===================== -->
+<joint name="joint3"
+       type="revolute">
+    <parent link="link2"/>
+    <child link="link3"/>
+    <origin xyz="0.35 0 0"/>
+    <axis xyz="0 1 0"/>
+    <limit
+        lower="-2.2"
+        upper="2.2"
+        effort="20"
+        velocity="1"/>
+</joint>
+<link name="link3">
+    <visual>
+        <geometry>
+            <box size="0.3 0.06 0.06"/>
         </geometry>
         <origin xyz="0.15 0 0"/>
     </visual>
 </link>
+<!-- ===================== -->
+<!-- Joint 4 Wrist rotate -->
+<!-- ===================== -->
+<joint name="joint4"
+       type="revolute">
+    <parent link="link3"/>
+    <child link="link4"/>
+    <origin xyz="0.3 0 0"/>
+    <axis xyz="1 0 0"/>
+    <limit
+        lower="-3.14"
+        upper="3.14"
+        effort="10"
+        velocity="1"/>
+</joint>
+<link name="link4">
+    <visual>
+        <geometry>
+            <cylinder radius="0.04"
+                      length="0.15"/>
+        </geometry>
+        <origin xyz="0 0 0.075"/>
+    </visual>
+</link>
+<!-- ===================== -->
+<!-- Joint 5 Wrist pitch -->
+<!-- ===================== -->
+<joint name="joint5"
+       type="revolute">
+    <parent link="link4"/>
+    <child link="link5"/>
+    <origin xyz="0 0 0.15"/>
+    <axis xyz="0 1 0"/>
+    <limit
+        lower="-1.57"
+        upper="1.57"
+        effort="10"
+        velocity="1"/>
+</joint>
+<link name="link5">
+    <visual>
+        <geometry>
+            <box size="0.15 0.06 0.06"/>
+        </geometry>
+        <origin xyz="0.075 0 0"/>
+    </visual>
+</link>
+<!-- ===================== -->
+<!-- Joint 6 Tool rotation -->
+<!-- ===================== -->
+<joint name="joint6"
+       type="revolute">
+    <parent link="link5"/>
+    <child link="tool_link"/>
+    <origin xyz="0.15 0 0"/>
+    <axis xyz="1 0 0"/>
+    <limit
+        lower="-3.14"
+        upper="3.14"
+        effort="10"
+        velocity="1"/>
+</joint>
+<link name="tool_link">
+    <visual>
+        <geometry>
+            <cylinder radius="0.04"
+                      length="0.1"/>
+        </geometry>
+        <origin xyz="0.05 0 0"/>
+    </visual>
+</link>
 </robot>

Commit message: complete day18 collision-aware planning and execution

File: ros2_ws/src/simple_6dof_description/urdf/simple_6dof_arm.urdf.xacro (robot description, xacro)
@@ -2,20 +2,24 @@
 <robot xmlns:xacro="http://www.ros.org/wiki/xacro"
        name="simple_6dof_arm">
-<!-- ===================== -->
-<!-- Base -->
-<!-- ===================== -->
-<link name="base_link">
-    <visual>
-        <geometry>
-            <box size="0.3 0.3 0.1"/>
-        </geometry>
-        <origin xyz="0 0 0"/>
-    </visual>
-</link>
-<!-- ===================== -->
-<!-- Joint 1 Base Rotation -->
-<!-- ===================== -->
-<joint name="joint1"
-       type="revolute">
+  <!-- ===================== -->
+  <!-- Base -->
+  <!-- ===================== -->
+  <link name="base_link">
+    <visual>
+      <geometry>
+        <box size="0.3 0.3 0.1"/>
+      </geometry>
+    </visual>
+    <collision>
+      <geometry>
+        <box size="0.3 0.3 0.1"/>
+      </geometry>
+    </collision>
+  </link>
+  <!-- ===================== -->
+  <!-- Joint 1 Base Rotation -->
+  <!-- ===================== -->
+  <joint name="joint1"
+         type="revolute">
     <parent link="base_link"/>
     <child link="link1"/>
@@ -23,23 +27,32 @@
     <axis xyz="0 0 1"/>
     <limit
-        lower="-3.14"
-        upper="3.14"
-        effort="20"
-        velocity="1"/>
-</joint>
-<link name="link1">
-    <visual>
-        <geometry>
-            <cylinder radius="0.05"
-                      length="0.35"/>
-        </geometry>
-        <origin xyz="0 0 0.175"/>
-    </visual>
-</link>
-<!-- ===================== -->
-<!-- Joint 2 Shoulder -->
-<!-- ===================== -->
-<joint name="joint2"
-       type="revolute">
+      lower="-3.14"
+      upper="3.14"
+      effort="20"
+      velocity="1"/>
+  </joint>
+  <link name="link1">
+    <visual>
+      <origin xyz="0 0 0.175"/>
+      <geometry>
+        <cylinder
+          radius="0.05"
+          length="0.35"/>
+      </geometry>
+    </visual>
+    <collision>
+      <origin xyz="0 0 0.175"/>
+      <geometry>
+        <cylinder
+          radius="0.05"
+          length="0.35"/>
+      </geometry>
+    </collision>
+  </link>
+  <!-- ===================== -->
+  <!-- Joint 2 Shoulder -->
+  <!-- ===================== -->
+  <joint name="joint2"
+         type="revolute">
     <parent link="link1"/>
     <child link="link2"/>
@@ -47,22 +60,28 @@
     <axis xyz="0 1 0"/>
     <limit
-        lower="-1.8"
-        upper="1.8"
-        effort="20"
-        velocity="1"/>
-</joint>
-<link name="link2">
-    <visual>
-        <geometry>
-            <box size="0.35 0.08 0.08"/>
-        </geometry>
-        <origin xyz="0.175 0 0"/>
-    </visual>
-</link>
-<!-- ===================== -->
-<!-- Joint 3 Elbow -->
-<!-- ===================== -->
-<joint name="joint3"
-       type="revolute">
+      lower="-1.8"
+      upper="1.8"
+      effort="20"
+      velocity="1"/>
+  </joint>
+  <link name="link2">
+    <visual>
+      <origin xyz="0.175 0 0"/>
+      <geometry>
+        <box size="0.35 0.08 0.08"/>
+      </geometry>
+    </visual>
+    <collision>
+      <origin xyz="0.175 0 0"/>
+      <geometry>
+        <box size="0.35 0.08 0.08"/>
+      </geometry>
+    </collision>
+  </link>
+  <!-- ===================== -->
+  <!-- Joint 3 Elbow -->
+  <!-- ===================== -->
+  <joint name="joint3"
+         type="revolute">
     <parent link="link2"/>
     <child link="link3"/>
@@ -70,22 +89,28 @@
     <axis xyz="0 1 0"/>
     <limit
-        lower="-2.2"
-        upper="2.2"
-        effort="20"
-        velocity="1"/>
-</joint>
-<link name="link3">
-    <visual>
-        <geometry>
-            <box size="0.3 0.06 0.06"/>
-        </geometry>
-        <origin xyz="0.15 0 0"/>
-    </visual>
-</link>
-<!-- ===================== -->
-<!-- Joint 4 Wrist rotate -->
-<!-- ===================== -->
-<joint name="joint4"
-       type="revolute">
+      lower="-2.2"
+      upper="2.2"
+      effort="20"
+      velocity="1"/>
+  </joint>
+  <link name="link3">
+    <visual>
+      <origin xyz="0.15 0 0"/>
+      <geometry>
+        <box size="0.3 0.06 0.06"/>
+      </geometry>
+    </visual>
+    <collision>
+      <origin xyz="0.15 0 0"/>
+      <geometry>
+        <box size="0.3 0.06 0.06"/>
+      </geometry>
+    </collision>
+  </link>
+  <!-- ===================== -->
+  <!-- Joint 4 Wrist Rotate -->
+  <!-- ===================== -->
+  <joint name="joint4"
+         type="revolute">
     <parent link="link3"/>
     <child link="link4"/>
@@ -93,23 +118,32 @@
     <axis xyz="1 0 0"/>
     <limit
-        lower="-3.14"
-        upper="3.14"
-        effort="10"
-        velocity="1"/>
-</joint>
-<link name="link4">
-    <visual>
-        <geometry>
-            <cylinder radius="0.04"
-                      length="0.15"/>
-        </geometry>
-        <origin xyz="0 0 0.075"/>
-    </visual>
-</link>
-<!-- ===================== -->
-<!-- Joint 5 Wrist pitch -->
-<!-- ===================== -->
-<joint name="joint5"
-       type="revolute">
+      lower="-3.14"
+      upper="3.14"
+      effort="10"
+      velocity="1"/>
+  </joint>
+  <link name="link4">
+    <visual>
+      <origin xyz="0 0 0.075"/>
+      <geometry>
+        <cylinder
+          radius="0.04"
+          length="0.15"/>
+      </geometry>
+    </visual>
+    <collision>
+      <origin xyz="0 0 0.075"/>
+      <geometry>
+        <cylinder
+          radius="0.04"
+          length="0.15"/>
+      </geometry>
+    </collision>
+  </link>
+  <!-- ===================== -->
+  <!-- Joint 5 Wrist Pitch -->
+  <!-- ===================== -->
+  <joint name="joint5"
+         type="revolute">
     <parent link="link4"/>
     <child link="link5"/>
@@ -117,22 +151,28 @@
     <axis xyz="0 1 0"/>
     <limit
-        lower="-1.57"
-        upper="1.57"
-        effort="10"
-        velocity="1"/>
-</joint>
-<link name="link5">
-    <visual>
-        <geometry>
-            <box size="0.15 0.06 0.06"/>
-        </geometry>
-        <origin xyz="0.075 0 0"/>
-    </visual>
-</link>
-<!-- ===================== -->
-<!-- Joint 6 Tool rotation -->
-<!-- ===================== -->
-<joint name="joint6"
-       type="revolute">
+      lower="-1.57"
+      upper="1.57"
+      effort="10"
+      velocity="1"/>
+  </joint>
+  <link name="link5">
+    <visual>
+      <origin xyz="0.075 0 0"/>
+      <geometry>
+        <box size="0.15 0.06 0.06"/>
+      </geometry>
+    </visual>
+    <collision>
+      <origin xyz="0.075 0 0"/>
+      <geometry>
+        <box size="0.15 0.06 0.06"/>
+      </geometry>
+    </collision>
+  </link>
+  <!-- ===================== -->
+  <!-- Joint 6 Tool Rotation -->
+  <!-- ===================== -->
+  <joint name="joint6"
+         type="revolute">
     <parent link="link5"/>
     <child link="tool_link"/>
@@ -140,17 +180,26 @@
     <axis xyz="1 0 0"/>
     <limit
-        lower="-3.14"
-        upper="3.14"
-        effort="10"
-        velocity="1"/>
-</joint>
-<link name="tool_link">
-    <visual>
-        <geometry>
-            <cylinder radius="0.04"
-                      length="0.1"/>
-        </geometry>
-        <origin xyz="0.05 0 0"/>
-    </visual>
-</link>
+      lower="-3.14"
+      upper="3.14"
+      effort="10"
+      velocity="1"/>
+  </joint>
+  <link name="tool_link">
+    <visual>
+      <origin xyz="0.05 0 0"/>
+      <geometry>
+        <cylinder
+          radius="0.04"
+          length="0.1"/>
+      </geometry>
+    </visual>
+    <collision>
+      <origin xyz="0.05 0 0"/>
+      <geometry>
+        <cylinder
+          radius="0.04"
+          length="0.1"/>
+      </geometry>
+    </collision>
+  </link>
 </robot>

Commit message: complete day20 gripper control

File: ros2_ws/src/simple_6dof_description/urdf/simple_6dof_arm.urdf.xacro (robot description, xacro)
@@ -203,3 +203,81 @@
     </collision>
   </link>
+  <!-- ===================== -->
+  <!-- Gripper Base          -->
+  <!-- ===================== -->
+  <joint name="gripper_mount_joint" type="fixed">
+    <parent link="tool_link"/>
+    <child link="gripper_base"/>
+    <origin xyz="0.10 0 0"/>
+  </joint>
+  <link name="gripper_base">
+    <visual>
+      <origin xyz="0.025 0 0"/>
+      <geometry>
+        <box size="0.05 0.12 0.08"/>
+      </geometry>
+    </visual>
+    <collision>
+      <origin xyz="0.025 0 0"/>
+      <geometry>
+        <box size="0.05 0.12 0.08"/>
+      </geometry>
+    </collision>
+  </link>
+  <!-- ===================== -->
+  <!-- Left Finger           -->
+  <!-- ===================== -->
+  <joint name="left_finger_joint" type="prismatic">
+    <parent link="gripper_base"/>
+    <child link="left_finger"/>
+    <origin xyz="0.05 0.06 0"/>
+    <axis xyz="0 1 0"/>
+    <limit
+      lower="0.0"
+      upper="0.04"
+      effort="20"
+      velocity="0.05"/>
+  </joint>
+  <link name="left_finger">
+    <visual>
+      <origin xyz="0.06 0 0"/>
+      <geometry>
+        <box size="0.12 0.02 0.03"/>
+      </geometry>
+    </visual>
+    <collision>
+      <origin xyz="0.06 0 0"/>
+      <geometry>
+        <box size="0.12 0.02 0.03"/>
+      </geometry>
+    </collision>
+  </link>
+  <!-- ===================== -->
+  <!-- Right Finger          -->
+  <!-- ===================== -->
+  <joint name="right_finger_joint" type="prismatic">
+    <parent link="gripper_base"/>
+    <child link="right_finger"/>
+    <origin xyz="0.05 -0.06 0"/>
+    <axis xyz="0 -1 0"/>
+    <limit
+      lower="0.0"
+      upper="0.04"
+      effort="20"
+      velocity="0.05"/>
+  </joint>
+  <link name="right_finger">
+    <visual>
+      <origin xyz="0.06 0 0"/>
+      <geometry>
+        <box size="0.12 0.02 0.03"/>
+      </geometry>
+    </visual>
+    <collision>
+      <origin xyz="0.06 0 0"/>
+      <geometry>
+        <box size="0.12 0.02 0.03"/>
+      </geometry>
+    </collision>
+  </link>
 </robot>

File: ros2_ws/src/simple_6dof_moveit_config/config/simple_6dof_arm.ros2_control.xacro (robot description, xacro)
@@ -50,4 +50,18 @@
                 <state_interface name="velocity"/>
             </joint>
+                        <joint name="left_finger_joint">
+                <command_interface name="position"/>
+                <state_interface name="position">
+                  <param name="initial_value">${initial_positions['left_finger_joint']}</param>
+                </state_interface>
+                <state_interface name="velocity"/>
+            </joint>
+            <joint name="right_finger_joint">
+                <command_interface name="position"/>
+                <state_interface name="position">
+                  <param name="initial_value">${initial_positions['right_finger_joint']}</param>
+                </state_interface>
+                <state_interface name="velocity"/>
+            </joint>
         </ros2_control>
     </xacro:macro>
